File: Smart_home.kicad_pcb (KiCad board)
At the start: 2 copper layers, 60 x 60 mm, 74 parts, among them J1 Screw_Terminal_01x02, J2 Screw_Terminal_01x04, J3 USB_C_Receptacle_USB2.0_16P, J4 Screw_Terminal_01x02, J5 Screw_Terminal_01x02, K1 G3MB-202PL, K2 G3MB-202PL, K3 G3MB-202PL, K4 G3MB-202PL, Q1 SS8050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

Commit message: Version v1.0 is ready for manufacturing.
Parts:
- added C11: 100nF, Capacitor_SMD:C_0603_1608Metric_Pad1.08x0.95mm_HandSolder, F.Cu at (165.6, 94.8)
- added C12: 100nF, Capacitor_SMD:C_0603_1608Metric_Pad1.08x0.95mm_HandSolder, F.Cu at (165.0, 100.8)
- added C13: 100nF, Capacitor_SMD:C_0603_1608Metric_Pad1.08x0.95mm_HandSolder, F.Cu at (159.8, 99.6)
- added C14: 100nF, Capacitor_SMD:C_0603_1608Metric_Pad1.08x0.95mm_HandSolder, F.Cu at (156.2, 99.6)
- added J6: Conn_01x05, Connector_JST:JST_XH_B5B-XH-A_1x05_P2.50mm_Vertical, F.Cu at (176.5, 99.2)
- added R25: 220, Resistor_SMD:R_0603_1608Metric_Pad0.98x0.95mm_HandSolder, F.Cu at (169.2, 99.2)
- added R26: 220, Resistor_SMD:R_0603_1608Metric_Pad0.98x0.95mm_HandSolder, F.Cu at (169.2, 101.0)
- added R27: 220, Resistor_SMD:R_0603_1608Metric_Pad0.98x0.95mm_HandSolder, F.Cu at (169.2, 102.8)
- added R28: 220, Resistor_SMD:R_0603_1608Metric_Pad0.98x0.95mm_HandSolder, F.Cu at (169.2, 104.5)
- added R29: 10K, Resistor_SMD:R_0805_2012Metric_Pad1.20x1.40mm_HandSolder, F.Cu at (165.8, 93.0)
- added R30: 10K, Resistor_SMD:R_0805_2012Metric_Pad1.20x1.40mm_HandSolder, F.Cu at (162.8, 98.6)
- added R31: 10K, Resistor_SMD:R_0805_2012Metric_Pad1.20x1.40mm_HandSolder, F.Cu at (159.8, 97.8)
- added R32: 10K, Resistor_SMD:R_0805_2012Metric_Pad1.20x1.40mm_HandSolder, F.Cu at (156.0, 97.8)
- added U5: 74HC14, Package_SO:SOIC-14_3.9x8.7mm_P1.27mm, B.Cu at (158.8, 79.5)
- added kibuzzard-6A2A5232: G***, kibuzzard-6A2A5232, F.Cu at (155.0, 103.6)
- added kibuzzard-6A2A52E4: G***, kibuzzard-6A2A52E4, F.Cu at (155.0, 105.4)
- moved J2 2.50 mm to (151.8, 114.5)
- renumbered J5 to J3, J3 to J4, J4 to J5
Routing:
- net +5V: track 121.8 -> 170.6 mm, vias 0 -> 2
- net Net-(C14-Pad1): track 0.00 -> 38.5 mm, vias 0 -> 1
- net Net-(C13-Pad1): track 0.00 -> 32.7 mm, vias 0 -> 1
- net /IO7: track 0.00 -> 29.2 mm, vias 0 -> 1
- net /IO10: track 0.00 -> 28.0 mm, vias 0 -> 1
- net Net-(C12-Pad1): track 0.00 -> 23.6 mm, vias 0 -> 1
- net /USB_D-/IO18: track 0.00 -> 20.4 mm, vias 0 -> 1
- net Net-(C11-Pad1): track 0.00 -> 20.0 mm, vias 0 -> 1
- net VUSB: track 35.3 -> 48.4 mm, vias 0 -> 4
- net /Input_buttons/BTN_{in}4: track 0.00 -> 7.36 mm
- net /Input_buttons/BTN_{in}3: track 0.00 -> 7.05 mm
- net /Input_buttons/BTN_{in}2: track 0.00 -> 6.74 mm
- net /Input_buttons/BTN_{in}1: track 0.00 -> 6.43 mm
- net /USB_D+/IO19: track 0.00 -> 3.97 mm, vias 0 -> 1
- net /LINE2: track 40.1 -> 36.2 mm
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Other:
- outline, holes or cut-outs redrawn
- board text added: "${REVISION}"
