File: Smart_home.kicad_sch (KiCad schematic)
At the start: 73 parts, among them J1 Screw_Terminal_01x02, J2 Screw_Terminal_01x04, J3 USB_C_Receptacle_USB2.0_16P, J4 Screw_Terminal_01x02, J5 Screw_Terminal_01x02, K1 G3MB-202PL, K2 G3MB-202PL, K3 G3MB-202PL, K4 G3MB-202PL, Q1 SS8050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

Commit message: Version v1.0 is ready for manufacturing.
Parts:
- renumbered J5 to J3, J3 to J4, J4 to J5
Connections:
- no-connect marks 15 -> 12
Other:
- added sheet Input_buttons (Input_buttons.kicad_sch)
- company: (none) -> U3 Co.
- title: (none) -> Smart Home System
- moved on the sheet: J5
